File: Drv_board.kicad_pcb (KiCad board)
At the start: 2 copper layers, 100 x 100 mm, 111 parts, among them IC1 TPS61087DRCR, IC2 DRV8836DSSR, J1 SRF-05_CONN, J10 U.FL, J2 OLED_CONN, J3 WS_LED_1_CONN, J4 USB_B_Micro, J5 QTR_CONN, J6 SWD, J7 WS_LED_0_CONN, J8 Motor A, J9 Motor B, Q1 DMP2045U, Q2 BC847-QR, SW1 SW_BOOT, U1 STM32F107RCTx, U2 USBLC6-2SC6, U3 MIC2288, U4 LD1117S50, U5 LD1117S33, U6 MPU-6050, U7 nRF24L01P, U8 M24C02-FMN, Y1 16 MHz, Y2 16 MHz

Commit message: done boost converter layout
Parts:
- BT1: footprint TerminalBlock_Phoenix:TerminalBlock_Phoenix_MKDS-1,5-2-5.08_1x02_P5.08mm_Horizontal -> TerminalBlock_Phoenix:TerminalBlock_Phoenix_PT-1,5-2-3.5-H_1x02_P3.50mm_Horizontal
- J6: footprint Connector_PinHeader_2.54mm:PinHeader_2x05_P2.54mm_Vertical -> Connector_PinHeader_2.00mm:PinHeader_2x05_P2.00mm_Vertical
- JP1: moved to B.Cu
- SW1: footprint Connector_PinHeader_1.00mm:PinHeader_1x03_P1.00mm_Vertical -> Connector_PinHeader_2.54mm:PinHeader_1x03_P2.54mm_Vertical
- moved U7 109.7 mm to (42.2, 166.3)
- moved D6 102.3 mm to (102.4, 138.7), turned to -90 degrees
- moved J1 100.7 mm to (41.8, 112.9)
- moved C26 95.9 mm to (103.8, 134.1)
- moved C27 93.0 mm to (103.8, 131.7)
- moved L1 92.1 mm to (127.1, 144.1)
- moved U3 91.4 mm to (128.4, 139.9), turned to 180 degrees
- moved C15 87.1 mm to (238.0, 51.5)
- moved C17 87.1 mm to (238.0, 56.5)
- moved C18 87.1 mm to (238.0, 59.0)
- moved C31 87.1 mm to (238.0, 86.1)
- moved C32 87.1 mm to (238.0, 88.6)
- moved C33 87.1 mm to (238.0, 91.1)
- moved C34 87.1 mm to (238.0, 93.6)
- moved C35 87.1 mm to (238.0, 96.1)
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Routing:
- net Net-(IC1-SS): track 0.00 -> 9.59 mm, vias 0 -> 2
- net 5V_Conv: track 0.00 -> 7.26 mm
- net +6V: track 0.00 -> 4.73 mm
- net Net-(IC1-FB): track 0.00 -> 4.50 mm
- net Net-(U3-FB): track 0.00 -> 3.85 mm
- net Net-(IC1-FREQ): track 0.00 -> 3.64 mm, vias 0 -> 1
- net Net-(D4-A): track 0.00 -> 3.51 mm
- net +BATT: track 0.00 -> 3.21 mm, vias 0 -> 1
- net Net-(IC1-COMP): track 0.00 -> 2.44 mm
- net Net-(C25-Pad1): track 0.00 -> 2.41 mm
- net Net-(D7-A): track 0.00 -> 2.21 mm
- net GND: track 0.00 -> 1.50 mm, vias 0 -> 11
- net EN: track 0.00 -> 1.50 mm, vias 0 -> 3
- net +3.3V: vias 0 -> 4
- added copper zone on F.Cu, net +3.3V
- added copper zone on F.Cu, net +6V
- added copper zone on F.Cu, net +BATT
- added copper zone on F.Cu, net 5V_Conv
- added copper zone on F.Cu, net EN
- added copper zone on F.Cu, net GND
- added copper zone on In1.Cu, net GND
- added copper zone on F.Cu, net Net-(D2-A)
- added copper zone on F.Cu, net Net-(D6-A)
- added copper zone on F.Cu, net Net-(IC1-FREQ)
- added copper zone on F.Cu, net Net-(IC1-SS)
Other:
- board size 100 x 100 mm -> 70 x 70 mm
- copper layers 2 -> 4

Commit message: working
Parts:
- C40: footprint Capacitor_SMD:C_1210_3225Metric -> Capacitor_SMD:C_0603_1608Metric
- moved JP2 144.2 mm to (138.6, 133.9)
- moved S3 136.8 mm to (154.1, 139.7)
- moved R11 131.4 mm to (147.8, 131.5)
- moved Q1 130.3 mm to (147.8, 134.8), turned to -90 degrees
- moved U7 127.9 mm to (149.0, 95.9)
- moved R12 126.5 mm to (152.1, 131.5)
- moved D5 125.4 mm to (156.3, 134.8), turned to -90 degrees
- moved Q2 124.3 mm to (152.1, 134.8), turned to -90 degrees
- moved R9 115.3 mm to (156.3, 131.5)
- moved U6 110.9 mm to (139.2, 92.0)
- moved J1 106.3 mm to (140.1, 72.5), turned to 180 degrees
- moved U8 104.5 mm to (148.8, 109.7)
- moved C2 103.6 mm to (134.5, 114.6), turned to 180 degrees
- moved J10 99.9 mm to (156.5, 90.7), turned to 90 degrees
- moved C4 99.3 mm to (138.7, 109.2), turned to 90 degrees
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Routing:
- net EN: track 1.50 -> 41.1 mm
- net V_USB: track 0.00 -> 18.8 mm
- net Net-(Q1-G): track 0.00 -> 12.2 mm
- net USB_D+: track 0.00 -> 11.9 mm
- net USB_D-: track 0.00 -> 11.9 mm
- net LATCH_POWERUP: track 0.00 -> 11.5 mm, vias 0 -> 1
- net Net-(D5-Pad3): track 0.00 -> 7.20 mm
- net USB_CONN_D-: track 0.00 -> 6.45 mm
- net USB_CONN_D+: track 0.00 -> 6.43 mm
- net Net-(D4-A): track 3.51 -> 8.66 mm
- net +6V: track 4.73 -> 0.00 mm
- net Net-(D7-A): track 2.21 -> 6.87 mm
- net GND: track 1.50 -> 6.14 mm, vias 11 -> 61
- net Power_Btn: track 0.00 -> 2.24 mm
- net Net-(Q2-B): track 0.00 -> 2.24 mm
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- added copper zone on In2.Cu, net +BATT
- added copper zone on F.Cu, net Net-(Q1-G)
- added copper zone on F.Cu, net V_USB
- removed copper zone on F.Cu, net Net-(IC1-FREQ)
Other:
- board size 70 x 70 mm -> 60 x 80 mm

Commit message: working on pcb
Parts:
- C11: renamed from C3; footprint Capacitor_SMD:C_0402_1005Metric -> Capacitor_SMD:C_0603_1608Metric
- C12: renamed from C6; footprint Capacitor_SMD:C_0402_1005Metric -> Capacitor_SMD:C_0603_1608Metric
- C31: renamed from C43; footprint Capacitor_SMD:C_0402_1005Metric -> Capacitor_SMD:C_0603_1608Metric
- C32: renamed from C44; footprint Capacitor_SMD:C_0402_1005Metric -> Capacitor_SMD:C_0603_1608Metric
- C38: renamed from C41; footprint Capacitor_SMD:C_0402_1005Metric -> Capacitor_SMD:C_0603_1608Metric
- C39: renamed from C42; footprint Capacitor_SMD:C_0402_1005Metric -> Capacitor_SMD:C_0603_1608Metric
- C40: renamed from C36; footprint Capacitor_SMD:C_0402_1005Metric -> Capacitor_SMD:C_0603_1608Metric
- C46: renamed from C38; footprint Capacitor_SMD:C_0402_1005Metric -> Capacitor_SMD:C_0603_1608Metric
- D1, D7: footprint LED_SMD:LED_0805_2012Metric -> LED_SMD:LED_0603_1608Metric
- D6: renamed from D4; footprint LED_SMD:LED_0805_2012Metric -> LED_SMD:LED_0603_1608Metric
- JP2: footprint Connector_PinHeader_2.54mm:PinHeader_1x03_P2.54mm_Vertical -> Jumper:SolderJumper-3_P1.3mm_Open_Pad1.0x1.5mm; moved to B.Cu
- L3: renamed from L4; footprint Inductor_SMD:L_0402_1005Metric -> Inductor_SMD:L_0603_1608Metric
- L4: renamed from L3; footprint Inductor_SMD:L_0402_1005Metric -> Inductor_SMD:L_0603_1608Metric
- L5: footprint Inductor_SMD:L_0402_1005Metric -> Inductor_SMD:L_0603_1608Metric
- S1, S2: footprint TL3305CF160QG:TL3305AF160QG -> digikey-footprints:Switch_Tactile_SMD_6x6mm_PTS645
- S3: value Power Up -> POWER UP; footprint TL3305CF160QG:TL3305AF160QG -> digikey-footprints:Switch_Tactile_SMD_6x6mm_PTS645
- SW1: footprint Connector_PinHeader_2.54mm:PinHeader_1x03_P2.54mm_Vertical -> Jumper:SolderJumper-3_P1.3mm_Open_Pad1.0x1.5mm
- moved R4 78.9 mm to (141.8, 90.7)
- moved C11 71.4 mm to (136.0, 88.8)
- moved Y1 70.6 mm to (131.7, 89.1), turned to 180 degrees
- moved C12 64.0 mm to (126.4, 89.5), turned to 180 degrees
- moved J8 56.9 mm to (103.9, 125.4), turned to 90 degrees
- moved J9 53.5 mm to (156.2, 117.9), turned to -90 degrees
- moved S1 33.0 mm to (154.2, 94.0)
- moved U7 32.0 mm to (116.8, 111.4)
- moved S3 30.6 mm to (154.2, 109.1)
- moved J7 25.0 mm to (113.5, 97.5), turned to 180 degrees
- moved U8 24.4 mm to (163.1, 87.2)
- moved C6 20.0 mm to (141.0, 104.9), turned to 180 degrees
- moved C2 19.8 mm to (138.9, 95.3), turned to -90 degrees
- moved C28 18.3 mm to (93.2, 115.1)
- moved S2 18.3 mm to (154.2, 101.6)
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- renumbered C9 to C10, C23 to C13, C21 to C14, C22 to C15, C26 to C16, C27 to C17, C16 to C18, C13 to C21, C14 to C22, C24 to C23, C25 to C24, C15 to C25, C17 to C26, C18 to C27, C4 to C3, C31 to C33, C32 to C34, C33 to C35, C45 to C36, C46 to C37, C5 to C4, C34 to C41, C35 to C42, C39 to C43, C40 to C44, C37 to C45, C7 to C5, C8 to C6, C10 to C7, C11 to C8, C12 to C9, D5 to D2, D6 to D4, D2 to D5, J4 to J1, J3 to J2, J7 to J3, J5 to J4, J1 to J5, J2 to J6, J6 to J7, JP3 to JP1, JP1 to JP3, L2 to L1, L1 to L2, R4 to R1, R14 to R10, R7 to R11, R10 to R12, R16 to R13, R15 to R14, R13 to R15, R8 to R16, R20 to R17, R17 to R18, R18 to R19, R3 to R2, R19 to R20, R2 to R3, R1 to R4, R9 to R5, R11 to R6, R5 to R7, R12 to R8, R6 to R9, U2 to U1, U1 to U2, U5 to U3, U3 to U4, U4 to U5, U7 to U6, U8 to U7, U6 to U8
Connections:
- J9 pad 1: B1 -> B2
- J9 pad 6: B2 -> B1
Routing:
- net USB_D+: track 11.9 -> 70.1 mm
- net USB_D-: track 11.9 -> 70.1 mm
- net A1: track 0.00 -> 32.1 mm
- net B1: track 0.00 -> 32.1 mm
- net B2: track 0.00 -> 25.0 mm
- net A2: track 0.00 -> 25.0 mm
- net DRV_NSLEEP: track 0.00 -> 24.0 mm
- net DRV_MODE: track 0.00 -> 23.9 mm
- net LATCH_POWERUP: track 11.5 -> 21.1 mm
- net DRV_AIN1/APHASE: track 0.00 -> 8.44 mm
- net DRV_BIN2/BENBL: track 0.00 -> 8.44 mm
- net DRV_BIN1/BPHASE: track 0.00 -> 8.44 mm
- net DRV_AIN2/AENBL: track 0.00 -> 8.44 mm
- net Net-(U2-PD0): track 0.00 -> 7.50 mm
- net Net-(U2-PD1): track 0.00 -> 4.66 mm
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- added copper zone on F.Cu, net A1
- added copper zone on F.Cu, net A2
- added copper zone on F.Cu, net B1
- added copper zone on F.Cu, net B2
- added copper zone on F.Cu, net Net-(D6-A)
- removed copper zone on F.Cu, net Net-(D4-A)
- removed copper zone on F.Cu, net Net-(Q1-G)

Commit message: more layout added
Parts:
- JP1: moved to B.Cu
- moved JP1 150.6 mm to (122.4, 124.2), turned to -90 degrees
- moved Y2 119.0 mm to (137.4, 82.0)
- moved C30 53.2 mm to (127.0, 116.6), turned to 90 degrees
- moved C29 51.5 mm to (125.2, 116.6), turned to 90 degrees
- moved U8 28.5 mm to (142.2, 106.7)
- moved C28 28.0 mm to (121.2, 113.8), turned to 0 degrees
- moved U7 23.9 mm to (116.8, 87.5)
- moved SW1 21.8 mm to (61.7, 93.2)
- moved C1 14.9 mm to (124.0, 91.9)
- moved C6 6.04 mm to (135.4, 107.2), turned to -90 degrees
- moved C11 3.66 mm to (133.2, 91.2)
- moved C12 3.53 mm to (129.5, 91.2)
- moved J10 3.21 mm to (157.2, 83.1), turned to -90 degrees
- moved J7 2.93 mm to (116.1, 96.1), turned to 0 degrees
- moved U6 2.34 mm to (145.4, 83.7)
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Connections:
- J8 pad 1: A1 -> A2
- J8 pad 6: A2 -> A1
- S3 pad 3: Net-(D2-Pad3) -> unconnected-(S3-Pad3)
Routing:
- net Net-(D2-Pad3): track 11.1 -> 34.9 mm
- net A1: track 32.1 -> 22.5 mm
- net B2: track 25.0 -> 31.7 mm
- net B1: track 32.1 -> 29.1 mm
- net DRV_NSLEEP: track 24.0 -> 21.5 mm
- net DRV_MODE: track 23.9 -> 21.5 mm
- net DRV_AIN2/AENBL: track 8.44 -> 6.25 mm
- net DRV_BIN2/BENBL: track 8.44 -> 6.25 mm
- net DRV_BIN1/BPHASE: track 8.44 -> 6.25 mm
- net DRV_AIN1/APHASE: track 8.44 -> 6.25 mm
- net GND: track 9.61 -> 10.6 mm
- net Net-(U2-PD0): track 7.50 -> 8.47 mm
- net Net-(U2-PD1): track 4.66 -> 5.63 mm
- net A2: track 25.0 -> 25.9 mm
- net 5V_Conv: vias 0 -> 5

Commit message: layout in progress
Parts:
- added REF**: PinHeader_2x08_P2.54mm_Vertical, Connector_PinHeader_2.54mm:PinHeader_2x08_P2.54mm_Vertical, F.Cu at (110.5, 85.3)
- C36, C37: footprint Capacitor_SMD:C_0402_1005Metric -> Capacitor_SMD:C_0603_1608Metric
- moved C25 146.5 mm to (110.0, 122.7)
- moved C43 131.7 mm to (111.3, 102.1)
- moved C26 130.1 mm to (126.0, 122.7)
- moved C27 129.9 mm to (126.0, 124.7)
- moved C44 127.6 mm to (111.3, 103.9)
- moved C40 108.0 mm to (137.7, 79.2), turned to 90 degrees
- moved R20 105.9 mm to (136.1, 93.2)
- moved R19 105.9 mm to (136.1, 91.4)
- moved L3 105.3 mm to (151.6, 82.5)
- moved L5 105.3 mm to (151.6, 84.6)
- moved L4 105.0 mm to (151.9, 80.8)
- moved C46 104.3 mm to (141.4, 95.6), turned to 180 degrees
- moved C36 103.7 mm to (142.2, 87.4), turned to 90 degrees
- moved C41 102.2 mm to (136.1, 100.7), turned to -90 degrees
- moved C37 97.9 mm to (148.3, 87.4), turned to -90 degrees
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Routing:
- net DRV_BIN2/BENBL: track 6.25 -> 20.7 mm
- net DRV_BIN1/BPHASE: track 6.25 -> 20.7 mm
- net DRV_AIN1/APHASE: track 6.25 -> 20.7 mm
- net DRV_AIN2/AENBL: track 6.25 -> 20.6 mm
- net USB_D-: track 69.9 -> 80.0 mm
- net USB_D+: track 69.8 -> 80.0 mm
- net DRV_MODE: track 21.5 -> 29.0 mm, vias 0 -> 2
- net B2: track 31.7 -> 24.8 mm
- net DRV_NSLEEP: track 21.5 -> 27.3 mm, vias 0 -> 2
- net A2: track 25.9 -> 29.0 mm
- net A1: track 22.5 -> 24.9 mm
- net Net-(U2-PD1): track 5.63 -> 4.62 mm
- net Net-(U2-PD0): track 8.47 -> 7.95 mm
Other:
- outline, holes or cut-outs redrawn

Commit message: more layout
Parts:
- moved R18 98.8 mm to (143.6, 79.0)
- moved J7 27.2 mm to (111.0, 107.0), turned to 0 degrees
- moved U7 24.8 mm to (137.3, 109.9)
- moved C43 23.1 mm to (134.4, 103.1), turned to 180 degrees
- moved C44 23.1 mm to (134.4, 104.9), turned to 180 degrees
- moved REF** 17.0 mm to (113.3, 102.1), turned to 180 degrees
- moved R19 12.6 mm to (136.9, 104.0), turned to 90 degrees
- moved R20 11.6 mm to (140.2, 104.0), turned to 90 degrees
- moved C41 10.4 mm to (146.4, 101.2)
- moved C33 9.68 mm to (140.5, 88.3)
- moved C45 8.02 mm to (146.4, 97.9), turned to -90 degrees
- moved L4 6.62 mm to (146.3, 84.3), turned to -90 degrees
- moved C1 6.27 mm to (121.9, 85.9)
- moved C31 5.45 mm to (151.6, 83.6), turned to 0 degrees
- moved R4 5.09 mm to (148.3, 96.5)
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Connections:
- J4 pad 10: unconnected-(J4-Pin_10-Pad10) -> QTR_CTRL
- J4 pad 3: QTR_CTRL -> unconnected-(J4-Pin_3-Pad3)
Routing:
- net SRF-05_IN: track 0.00 -> 47.7 mm, vias 0 -> 1
- net SRF-05_ECHO: track 0.00 -> 44.5 mm, vias 0 -> 1
- net GND: track 10.5 -> 54.3 mm, vias 57 -> 102
- net SRF-05_TRIG: track 0.00 -> 43.4 mm, vias 0 -> 1
- net +3.3V: track 0.00 -> 43.1 mm, vias 4 -> 16
- net I2C_SDA: track 0.00 -> 35.9 mm
- net I2C_SCL: track 0.00 -> 33.7 mm
- net QTR_CTRL: track 0.00 -> 31.2 mm, vias 0 -> 1
- net QTR_4: track 0.00 -> 27.2 mm, vias 0 -> 1
- net QTR_5: track 0.00 -> 25.6 mm, vias 0 -> 1
- net QTR_0: track 0.00 -> 24.8 mm, vias 0 -> 1
- net QTR_2: track 0.00 -> 24.6 mm, vias 0 -> 1
- net NRF_SCK: track 0.00 -> 22.8 mm, vias 0 -> 2
- net QTR_3: track 0.00 -> 22.7 mm, vias 0 -> 1
- net NRF_CSN: track 0.00 -> 21.2 mm
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- added copper zone on B.Cu, net GND

Commit message: layout
Parts:
- moved J7 35.6 mm to (141.3, 125.7), turned to 90 degrees
- moved REF** 9.92 mm to (113.3, 112.0)
Routing:
- net GND: vias 102 -> 98
- net +BATT: vias 15 -> 6

Commit message: layout...
Parts:
- moved R12 19.4 mm to (143.0, 128.8)
- moved D7 19.0 mm to (96.6, 128.3)
- moved D6 17.4 mm to (134.6, 124.5)
- moved C19 15.8 mm to (140.6, 131.7), turned to 0 degrees
- moved C20 14.0 mm to (137.0, 131.7), turned to 180 degrees
- moved R13 12.8 mm to (96.5, 131.2)
- moved D1 12.3 mm to (93.5, 50.3)
- moved J7 11.8 mm to (145.5, 114.7), turned to 180 degrees
- moved JP1 10.9 mm to (111.5, 124.5)
- moved U3 10.6 mm to (138.8, 137.0), turned to -90 degrees
- moved C25 10.5 mm to (116.6, 130.8), turned to 90 degrees
- moved U5 9.48 mm to (121.4, 132.5), turned to -90 degrees
- moved C26 7.75 mm to (119.6, 127.1), turned to 180 degrees
- moved REF** 7.13 mm to (113.3, 104.9)
- moved C27 3.68 mm to (123.2, 127.1)
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Routing:
- net NRST: track 0.00 -> 30.9 mm, vias 0 -> 1
- net SWO: track 0.00 -> 24.0 mm, vias 0 -> 1
- net SWDIO: track 0.00 -> 23.8 mm
- net SWCLK: track 0.00 -> 23.4 mm, vias 0 -> 1
- net Net-(D6-A): track 8.66 -> 0.00 mm
- net Net-(D7-A): track 6.87 -> 0.00 mm
- net GND: track 54.3 -> 58.7 mm, vias 98 -> 74
- net DRV_BIN1/BPHASE: track 17.5 -> 20.3 mm
- net DRV_AIN1/APHASE: track 17.5 -> 20.3 mm
- net DRV_NSLEEP: track 24.8 -> 27.6 mm
- net DRV_BIN2/BENBL: track 17.5 -> 20.3 mm
- net DRV_AIN2/AENBL: track 17.5 -> 20.3 mm
- net DRV_MODE: track 27.1 -> 29.7 mm
- net 5V_Conv: track 5.46 -> 3.65 mm, vias 5 -> 0
- net V_USB: track 18.8 -> 20.5 mm
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- added copper zone on F.Cu, net 5V_Stab
