File: Drv_board.kicad_pcb (KiCad board)
At the start: 4 copper layers, 60 x 80 mm, 112 parts, among them IC1 TPS61087DRCR, IC2 DRV8836DSSR, J1 USB_B_Micro, J10 U.FL, J2 WS_LED_1_CONN, J3 WS_LED_0_CONN, J4 QTR_CONN, J5 SRF-05_CONN, J6 OLED_CONN, J7 SWD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

Commit message: layout
Parts:
- moved C10 81.4 mm to (132.5, 89.5), turned to 90 degrees
- moved R2 78.2 mm to (134.4, 89.5), turned to -90 degrees
- moved R1 70.2 mm to (89.7, 98.6)
- moved R4 13.4 mm to (154.2, 108.6), turned to 0 degrees
- moved REF** 7.37 mm to (113.3, 112.3)
- moved C3 3.04 mm to (130.6, 87.9)
- moved JP2 2.34 mm to (135.6, 137.9)
- moved C12 1.78 mm to (124.2, 88.6)
- moved Y1 1.78 mm to (126.2, 85.8)
- moved C11 1.78 mm to (128.0, 88.6)
- moved S3 1.37 mm to (154.2, 113.0)
- moved S1 1.27 mm to (154.2, 95.2)
- moved C36 1.26 mm to (140.8, 92.1)
- moved C37 1.26 mm to (147.4, 92.1)
- moved Y2 1.26 mm to (144.1, 92.1)
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Routing:
- net KEEP_ALIVE: track 0.00 -> 74.0 mm, vias 0 -> 2
- net Power_Btn: track 2.24 -> 58.8 mm, vias 0 -> 2
- net Net-(U2-PC15): track 0.00 -> 53.3 mm, vias 0 -> 2
- net NRST: track 30.9 -> 51.3 mm
- net +BATT: track 3.66 -> 12.0 mm
- net LATCH_POWERUP: track 21.1 -> 25.5 mm
- net +3.3V: track 42.8 -> 44.9 mm, vias 18 -> 21
- net GND: track 58.7 -> 60.7 mm, vias 74 -> 76
- net EN: track 39.9 -> 38.0 mm
- net Net-(D2-Pad3): track 32.4 -> 31.0 mm
- net SRF-05_TRIG: track 43.4 -> 42.1 mm
- net NRF_XC1: track 6.37 -> 7.59 mm
- net NRF_XC2: track 8.91 -> 9.92 mm
- net Net-(U2-PD1): track 4.99 -> 5.95 mm
- net +3.3VA: track 7.68 -> 8.58 mm
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
Commit message: layout...
Parts:
- removed REF**: PinHeader_2x08_P2.54mm_Vertical, Connector_PinHeader_2.54mm:PinHeader_2x08_P2.54mm_Vertical
- added J11: BREAKOUT, Connector_PinHeader_2.54mm:PinHeader_2x07_P2.54mm_Vertical, F.Cu at (111.0, 101.1)
- moved D6 41.3 mm to (175.7, 127.8)
- moved R12 27.9 mm to (170.9, 128.0)
- moved JP1 14.5 mm to (97.2, 122.7)
- moved C1 8.10 mm to (128.4, 82.5)
- moved C26 8.05 mm to (127.6, 127.9), turned to -90 degrees
- moved C27 6.28 mm to (129.4, 127.9), turned to -90 degrees
- moved FB1 4.25 mm to (119.5, 84.6)
- moved C9 3.91 mm to (121.3, 84.6), turned to -90 degrees
- moved BT1 3.05 mm to (135.6, 143.6)
- moved J1 3.05 mm to (147.1, 144.1)
- moved C13 2.78 mm to (115.1, 136.9)
- moved C14 2.78 mm to (118.9, 141.1)
- moved C15 2.78 mm to (120.7, 141.1)
- moved C16 2.78 mm to (104.4, 134.1)
- moved C17 2.78 mm to (104.4, 131.8)
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Connections:
- J4 pad 10: QTR_CTRL -> QTR_1
- J4 pad 3: unconnected-(J4-Pin_3-Pad3) -> QTR_CTRL
- J4 pad 4: QTR_0 -> unconnected-(J4-Pin_4-Pad4)
- J4 pad 5: QTR_1 -> QTR_4
- J4 pad 6: QTR_2 -> QTR_5
- J4 pad 7: QTR_3 -> QTR_2
- J4 pad 8: QTR_4 -> QTR_3
- J4 pad 9: QTR_5 -> QTR_0
- S1 pad 4: NRST -> unconnected-(S1-Pad4)
- U2 pad 10: unconnected-(U2-PC2-Pad10) -> EXT_PC2
- U2 pad 11: unconnected-(U2-PC3-Pad11) -> EXT_PC3
- U2 pad 16: unconnected-(U2-PA2-Pad16) -> EXT_USART_TX
- U2 pad 17: unconnected-(U2-PA3-Pad17) -> EXT_USART_RX
- U2 pad 20: unconnected-(U2-PA4-Pad20) -> EXT_PA4
- U2 pad 34: unconnected-(U2-PB13-Pad34) -> EXT_SPI_SCK
- U2 pad 35: unconnected-(U2-PB14-Pad35) -> EXT_SPI_MISO
- U2 pad 36: unconnected-(U2-PB15-Pad36) -> EXT_SPI_MOSI
Routing:
- net ENC_B_2: track 0.00 -> 49.6 mm, vias 0 -> 1
- net ENC_B_1: track 0.00 -> 48.7 mm, vias 0 -> 1
- net WS_LED_0: track 0.00 -> 47.0 mm, vias 0 -> 2
- net ENC_A_2: track 0.00 -> 44.1 mm, vias 0 -> 1
- net ENC_A_1: track 0.08 -> 42.2 mm, vias 0 -> 1
- net I2C_SCL: track 33.7 -> 74.3 mm, vias 0 -> 2
- net I2C_SDA: track 35.9 -> 75.5 mm, vias 0 -> 2
- net WS_LED_1: track 0.00 -> 37.6 mm, vias 0 -> 1
- net EXT_USART_TX: track 0.00 -> 23.7 mm, vias 0 -> 2
- net EXT_PC3: track 0.00 -> 23.7 mm
- net EXT_USART_RX: track 0.00 -> 22.8 mm, vias 0 -> 2
- net EXT_PC2: track 0.00 -> 21.8 mm
- net EXT_SPI_MISO: track 0.00 -> 19.8 mm
- net EXT_SPI_MOSI: track 0.00 -> 17.6 mm
- net GND: track 60.7 -> 77.3 mm, vias 76 -> 79
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Other:
- board size 60 x 80 mm -> 60 x 77 mm

Commit message: layout finalising
Parts:
- J11: footprint Connector_PinHeader_2.54mm:PinHeader_2x07_P2.54mm_Vertical -> Connector_PinHeader_2.54mm:PinHeader_2x08_P2.54mm_Vertical
- SW1: moved to B.Cu
- moved R9 156.2 mm to (103.6, 115.7)
- moved R7 154.1 mm to (107.1, 115.7)
- moved SW1 83.4 mm to (141.1, 118.7), turned to 180 degrees
- moved R3 74.5 mm to (135.8, 81.4), turned to 90 degrees
- moved R1 52.4 mm to (141.1, 108.6), turned to -90 degrees
- moved D1 51.0 mm to (133.9, 81.4), turned to -90 degrees
- moved JP1 37.4 mm to (134.0, 128.9), turned to 0 degrees
- moved D6 28.0 mm to (147.7, 127.3), turned to 180 degrees
- moved R12 26.5 mm to (144.4, 127.3), turned to 0 degrees
- moved R13 18.7 mm to (114.9, 128.0), turned to 90 degrees
- moved D7 15.8 mm to (112.4, 127.3), turned to 0 degrees
- moved C1 3.00 mm to (130.6, 84.6), turned to -90 degrees
- moved C7 1.60 mm to (119.7, 87.9)
- moved C8 1.60 mm to (117.9, 87.8)
- moved C9 1.60 mm to (119.7, 84.6)
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Connections:
- J11 pad 3: WS_LED_1 -> KEEP_ALIVE
- J11 pad 4: WS_LED_0 -> Power_Btn
- R12 pad 1: 5V_Conv -> +3.3V
Routing:
- net BATT_ADC_0: track 0.00 -> 38.6 mm, vias 0 -> 2
- net EXT_PA4: track 0.00 -> 28.1 mm, vias 0 -> 2
- net Net-(D1-K): track 0.00 -> 24.0 mm
- net +BATT: track 12.0 -> 35.2 mm, vias 6 -> 7
- net NRF_IRQ: track 0.00 -> 22.7 mm
- net KEEP_ALIVE: track 71.5 -> 93.7 mm, vias 2 -> 4
- net BOOT0: track 0.00 -> 20.4 mm, vias 0 -> 2
- net Power_Btn: track 55.7 -> 74.4 mm, vias 2 -> 3
- net GND: track 77.3 -> 95.2 mm, vias 79 -> 91
- net +5V: track 0.00 -> 17.6 mm, vias 0 -> 4
- net WS_LED_1: track 37.6 -> 24.5 mm
- net WS_LED_0: track 47.0 -> 34.5 mm
- net +3.3V: track 41.6 -> 53.2 mm, vias 19 -> 22
- net Net-(SW1-B): track 0.00 -> 9.35 mm, vias 0 -> 1
- net 5V_Stab: track 9.94 -> 13.4 mm, vias 6 -> 4
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- added copper zone on In2.Cu, net +3.3V
- added copper zone on B.Cu, net +5V
- added copper zone on In2.Cu, net +5V
- added copper zone on In2.Cu, net +6V
- added copper zone on B.Cu, net 5V_Conv
- added copper zone on B.Cu, net 5V_Stab
- added copper zone on F.Cu, net Net-(D4-A)
- removed copper zone on F.Cu, net Net-(D6-A)

Commit message: layout completed
Parts:
- added TP1: Test MOSI, TestPoint:TestPoint_Pad_D1.0mm, B.Cu at (140.5, 84.5)
- added TP2: Test MISO, TestPoint:TestPoint_Pad_D1.0mm, B.Cu at (137.0, 86.7)
- added TP3: Test SCK, TestPoint:TestPoint_Pad_D1.0mm, B.Cu at (137.0, 84.5)
- added TP4: Test CSN, TestPoint:TestPoint_Pad_D1.0mm, B.Cu at (140.5, 82.2)
- added TP5: Test CE, TestPoint:TestPoint_Pad_D1.0mm, B.Cu at (137.0, 82.2)
- added TP6: Test IRQ, TestPoint:TestPoint_Pad_D1.0mm, B.Cu at (140.5, 86.7)
- moved R4 3.62 mm to (150.6, 108.6)
- moved C36 1.32 mm to (139.7, 91.4)
- moved C37 1.32 mm to (146.3, 91.4)
- moved Y2 1.32 mm to (143.0, 91.4)
- moved R3 0.90 mm to (135.1, 82.0)
- moved D1 0.90 mm to (133.2, 82.0)
- moved JP1 0.76 mm to (133.2, 128.9)
- moved BT1 0.38 mm to (135.6, 143.2)
- moved R7 0.38 mm to (107.1, 116.1)
- moved R9 0.38 mm to (103.6, 116.1)
- moved J5 0.25 mm to (138.3, 72.6)
- moved C14 0.19 mm to (118.9, 140.9)
- moved C15 0.19 mm to (120.7, 140.9)
- moved C21 0.14 mm to (126.8, 143.5)
- moved J1 0.13 mm to (147.1, 144.0)
Routing:
- net MPU-6050_IRQ: track 3.40 -> 19.1 mm, vias 1 -> 2
- net unconnected-(J1-Shield-Pad6): track 0.00 -> 9.16 mm
- net +3.3V: track 53.2 -> 61.0 mm, vias 22 -> 26
- net BOOT0: track 20.4 -> 24.1 mm
- net B1: track 28.2 -> 31.2 mm
- net A2: track 28.2 -> 31.2 mm
- net NRF_CSN: track 21.2 -> 23.9 mm, vias 0 -> 1
- net NRF_CE: track 20.9 -> 23.6 mm, vias 0 -> 1
- net Net-(U8-CPOUT): track 0.00 -> 2.02 mm
- net NRF_MISO: track 21.1 -> 23.0 mm, vias 0 -> 1
- net KEEP_ALIVE: track 93.7 -> 91.9 mm, vias 4 -> 3
- net NRF_MOSI: track 21.1 -> 22.9 mm, vias 0 -> 1
- net GND: track 95.2 -> 96.8 mm, vias 91 -> 130
- net NRF_SCK: track 22.8 -> 24.3 mm, vias 2 -> 3
- net NRF_IRQ: track 22.7 -> 24.2 mm, vias 0 -> 1
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Other:
- board text added: "+"
- board text added: "3.3V"
- board text added: "5V Src"
- board text added: "6V"
- board text added: "B.Freq"
- board text added: "Boot"
- board text added: "CE"
- board text added: "CSN"
- board text added: "DISP"
- board text added: "FUNCTION"
- board text added: "GPIO"
- board text added: "IRQ"
- board text added: "MISO"
- board text added: "MOSI"
- board text added: "MOTOR A"
- board text added: "MOTOR B"
- board text added: "POWER"
- board text added: "Powerup"
- board text added: "QTR"
- board text added: "RESET"
- board text added: "SCK"
- board text added: "SRF"
- board text added: "SWD"
- board text added: "USB"
- board text added: "WS 1"
- board text added: "WS 2"

Commit message: Completed PCB v1.0
Parts:
- JP1, JP2, JP3, SW1: footprint Jumper:SolderJumper-3_P1.3mm_Open_Pad1.0x1.5mm -> Jumper:SolderJumper-3_P1.3mm_Open_RoundedPad1.0x1.5mm
- S1, S2, S3: footprint digikey-footprints:Switch_Tactile_SMD_6x6mm_PTS645 -> digikey-footprints:Switch_Tactile_SMD_6x6mm
- moved SW1 4.89 mm to (137.4, 115.6)
- moved S1 0.25 mm to (153.9, 95.2)
- moved S2 0.25 mm to (153.9, 104.1)
- moved S3 0.25 mm to (153.9, 113.0)
Routing:
- net Net-(U2-PC15): track 51.3 -> 58.9 mm
- net NRST: track 48.2 -> 54.4 mm
- net Net-(SW1-B): track 9.35 -> 8.70 mm
Other:
- board text added: "Designed by M.Klebokowski"
- board text added: "JLCJLCJLCJLC"
- board text added: "Klebot"
- board text added: "Klebot rev 1.0 - 10/23"
